File: KiCAD/PowerPCB/PowerPCB.kicad_sch (KiCad schematic)
At the start: 12 parts, among them J1 GPIO, J2 Power In, J5 Serial, J6 Fan, Q1 DMMT5401, Q2 IRLML6401, Q3 IRLML6344

Commit message: Update PCBLayout
Parts:
- removed J1: GPIO, Connector_PinSocket_2.54mm:PinSocket_2x05_P2.54mm_Vertical, symbol Connector_Generic:Conn_02x05_Odd_Even
- removed J5: Serial, Connector_JST:JST_XH_B2B-XH-A_1x02_P2.50mm_Vertical, symbol Connector_Generic:Conn_01x02
- removed Q1: DMMT5401, Package_TO_SOT_SMD:SOT-23-6, symbol pixeltrace:DMMT5401
- removed Q2: IRLML6401, Package_TO_SOT_SMD:SOT-23, symbol pixeltrace:IRLML6401
- removed R1: 10k, Resistor_SMD:R_0805_2012Metric, symbol Device:R
- removed R2: 47k, Resistor_SMD:R_0805_2012Metric, symbol Device:R
- added J1: GPIO, Connector_PinSocket_2.54mm:PinSocket_2x06_P2.54mm_Vertical, symbol Connector_Generic:Conn_02x06_Odd_Even
- added J3: 5V Pad, TestPoint:TestPoint_THTPad_1.5x1.5mm_Drill0.7mm, symbol Connector:Conn_01x01_Pin
- R3, R4: footprint Resistor_SMD:R_0805_2012Metric -> Resistor_SMD:R_0805_2012Metric_Pad1.20x1.40mm_HandSolder
- renumbered J6 to J4
Connections:
- net 5V_IN is gone; now on net +5V: J2.1 (Pin_1)
- net +3V3: now also J1.1 (Pin_1)
- net +5V: now also J1.2 (Pin_2), J1.4 (Pin_4), J3.1 (Pin_1)
- net GND: now also J1.6 (Pin_6), J1.9 (Pin_9)
- net GPIO14/TXD0: now also J1.8 (Pin_8)
- net GPIO15/RXD0: now also J1.10 (Pin_10)
- net GPIO2/SDA1: now also J1.3 (Pin_3); no longer J2.2 (Pin_2)
- net GPIO3/SCL1: now also J1.5 (Pin_5)
- net GPIO4/GPCLK0: now also J1.7 (Pin_7); no longer R4.1
- new net GPIO17: J1.11 (Pin_11), J2.2 (Pin_2)
- new net GPIO18: J1.12 (Pin_12), R4.1
Other:
- note removed: "5V Powered HAT Protection"
- note removed: "Serial"
- moved on the sheet: D1, J4, Q3, R3, R4
